File: Hardware/Schematic/AnalogFrontend.sch (KiCad schematic (older format))
At the start: 10 parts, among them U2 MCP6L92

Commit message: Kicad v5 files added.
Parts:
- C11, C13, C3: symbol Ultrasonic-Flow-Sensor-rescue:C-Ultrasonic-Flow-Sensor-rescue-Ultrasonic-Flow-Sensor-rescue -> Ultrasonic-Flow-Sensor-rescue:C-Ultrasonic-Flow-Sensor-rescue-Ultrasonic-Flow-Sensor-rescue-Ultrasonic-Flow-Sensor-resc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
- R6, R9: symbol Ultrasonic-Flow-Sensor-rescue:R_Precision-res_precision-Ultrasonic-Flow-Sensor-rescue -> Ultrasonic-Flow-Sensor-rescue:R_Precision-res_precision-Ultrasonic-Flow-Sensor-rescue-Ultrasonic-Flow-Sensor-rescue
Changed lines of the file:
@@
-EESchema Schematic File Version 5
-EELAYER 33 0
+EESchema Schematic File Version 4
+EELAYER 30 0
 EELAYER END
 $Descr A4 11693 8268
 encoding utf-8
-Sheet 6 7
+Sheet 2 7
 Title ""
 Date ""
@@
 Comment3 ""
 Comment4 ""
-Comment5 ""
-Comment6 ""
-Comment7 ""
-Comment8 ""
-Comment9 ""
 $EndDescr
 Connection ~ 5550 4150
@@
 $EndComp
 $Comp
-L Ultrasonic-Flow-Sensor-rescue:R_Precision-res_precision-Ultrasonic-Flow-Sensor-rescue R6
+L Ultrasonic-Flow-Sensor-rescue:R_Precision-res_precision-Ultrasonic-Flow-Sensor-rescue-Ultrasonic-Flow-Sensor-rescue R6
 U 1 1 58F2F446
 P 4625 2500
@@
 $EndComp
 $Comp
-L Ultrasonic-Flow-Sensor-rescue:R_Precision-res_precision-Ultrasonic-Flow-Sensor-rescue R9
+L Ultrasonic-Flow-Sensor-rescue:R_Precision-res_precision-Ultrasonic-Flow-Sensor-rescue-Ultrasonic-Flow-Sensor-rescue R9
 U 1 1 5EAAE11D
 P 4625 4250
@@
 $EndComp
 $Comp
-L Ultrasonic-Flow-Sensor-rescue:C-Ultrasonic-Flow-Sensor-rescue-Ultrasonic-Flow-Sensor-rescue C3
+L Ultrasonic-Flow-Sensor-rescue:C-Ultrasonic-Flow-Sensor-rescue-Ultrasonic-Flow-Sensor-rescue-Ultrasonic-Flow-Sensor-rescue-Ultrasonic-Flow-Sensor-rescue C3
 U 1 1 58EC8D7E
 P 5175 3075
@@
 $EndComp
 $Comp
-L Ultrasonic-Flow-Sensor-rescue:C-Ultrasonic-Flow-Sensor-rescue-Ultrasonic-Flow-Sensor-rescue C11
+L Ultrasonic-Flow-Sensor-rescue:C-Ultrasonic-Flow-Sensor-rescue-Ultrasonic-Flow-Sensor-rescue-Ultrasonic-Flow-Sensor-rescue-Ultrasonic-Flow-Sensor-rescue C11
 U 1 1 5EA56652
 P 6000 2600
@@
 $EndComp
 $Comp
-L Ultrasonic-Flow-Sensor-rescue:C-Ultrasonic-Flow-Sensor-rescue-Ultrasonic-Flow-Sensor-rescue C13
+L Ultrasonic-Flow-Sensor-rescue:C-Ultrasonic-Flow-Sensor-rescue-Ultrasonic-Flow-Sensor-rescue-Ultrasonic-Flow-Sensor-rescue-Ultrasonic-Flow-Sensor-rescue C13
 U 1 1 5EA3DE50
 P 6000 4350
