File: Hardware/Schematic/Mcu.sch (KiCad schematic (older format))
At the start: 10 parts, among them J1 Conn_01x04_Male, U3 STM32F070F6Px, Y1 8MHz

Commit message: Kicad v5 files added.
Parts:
- C10, C8: symbol Ultrasonic-Flow-Sensor-rescue:C_Precision-cap_precision-Ultrasonic-Flow-Sensor-rescue -> Ultrasonic-Flow-Sensor-rescue:C_Precision-cap_precision-Ultrasonic-Flow-Sensor-rescue-Ultrasonic-Flow-Sensor-rescue
- C12, C15, C16: symbol Ultrasonic-Flow-Sensor-rescue:C-Ultrasonic-Flow-Sensor-rescue-Ultrasonic-Flow-Sensor-rescue -> Ultrasonic-Flow-Sensor-rescue:C-Ultrasonic-Flow-Sensor-rescue-Ultrasonic-Flow-Sensor-rescue-Ultrasonic-Flow-Sensor-resc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
- R3: symbol Ultrasonic-Flow-Sensor-rescue:R-Ultrasonic-Flow-Sensor-rescue-Ultrasonic-Flow-Sensor-rescue -> Ultrasonic-Flow-Sensor-rescue:R-Ultrasonic-Flow-Sensor-rescue-Ultrasonic-Flow-Sensor-rescue-Ultrasonic-Flow-Sensor-resc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
Changed lines of the file:
@@
-EESchema Schematic File Version 5
-EELAYER 33 0
+EESchema Schematic File Version 4
+EELAYER 30 0
 EELAYER END
 $Descr A4 11693 8268
 encoding utf-8
-Sheet 3 7
+Sheet 4 7
 Title ""
 Date ""
@@
 Comment3 ""
 Comment4 ""
-Comment5 ""
-Comment6 ""
-Comment7 ""
-Comment8 ""
-Comment9 ""
 $EndDescr
 Connection ~ 5600 2925
@@
 $EndComp
 $Comp
-L Ultrasonic-Flow-Sensor-rescue:R-Ultrasonic-Flow-Sensor-rescue-Ultrasonic-Flow-Sensor-rescue R3
+L Ultrasonic-Flow-Sensor-rescue:R-Ultrasonic-Flow-Sensor-rescue-Ultrasonic-Flow-Sensor-rescue-Ultrasonic-Flow-Sensor-rescue-Ultrasonic-Flow-Sensor-rescue R3
 U 1 1 58F39F96
 P 4800 3375
@@
 $EndComp
 $Comp
-L Ultrasonic-Flow-Sensor-rescue:C_Precision-cap_precision-Ultrasonic-Flow-Sensor-rescue C10
+L Ultrasonic-Flow-Sensor-rescue:C_Precision-cap_precision-Ultrasonic-Flow-Sensor-rescue-Ultrasonic-Flow-Sensor-rescue C10
 U 1 1 58F378A3
 P 4350 3825
@@
 $EndComp
 $Comp
-L Ultrasonic-Flow-Sensor-rescue:C_Precision-cap_precision-Ultrasonic-Flow-Sensor-rescue C8
+L Ultrasonic-Flow-Sensor-rescue:C_Precision-cap_precision-Ultrasonic-Flow-Sensor-rescue-Ultrasonic-Flow-Sensor-rescue C8
 U 1 1 5EAD11F0
 P 4350 4225
@@
 $EndComp
 $Comp
-L Ultrasonic-Flow-Sensor-rescue:C-Ultrasonic-Flow-Sensor-rescue-Ultrasonic-Flow-Sensor-rescue C12
+L Ultrasonic-Flow-Sensor-rescue:C-Ultrasonic-Flow-Sensor-rescue-Ultrasonic-Flow-Sensor-rescue-Ultrasonic-Flow-Sensor-rescue-Ultrasonic-Flow-Sensor-rescue C12
 U 1 1 58F0D0FE
 P 4800 3175
@@
 $EndComp
 $Comp
-L Ultrasonic-Flow-Sensor-rescue:C-Ultrasonic-Flow-Sensor-rescue-Ultrasonic-Flow-Sensor-rescue C16
+L Ultrasonic-Flow-Sensor-rescue:C-Ultrasonic-Flow-Sensor-rescue-Ultrasonic-Flow-Sensor-rescue-Ultrasonic-Flow-Sensor-rescue-Ultrasonic-Flow-Sensor-rescue C16
 U 1 1 58EC4449
 P 5300 2925
@@
 $EndComp
 $Comp
-L Ultrasonic-Flow-Sensor-rescue:C-Ultrasonic-Flow-Sensor-rescue-Ultrasonic-Flow-Sensor-rescue C15
+L Ultrasonic-Flow-Sensor-rescue:C-Ultrasonic-Flow-Sensor-rescue-Ultrasonic-Flow-Sensor-rescue-Ultrasonic-Flow-Sensor-rescue-Ultrasonic-Flow-Sensor-rescue C15
 U 1 1 5EA972CB
 P 5800 2925
